File: hardware/crommeter/crommeter.kicad_sch (KiCad schematic)
At the start: 0 parts

Commit message: Initial KiCad schematic done
Parts:
- added C1: 0.1uF, symbol Device:C
- added C2: 1uF, symbol Device:C
- added D1, D2, D3, D4, D5, D6, D7, D8: CUW_Y3SH.B2-GFJD-5J6T-Z242-20-R18-Z, CUW_Y3SH.B2-GFJD-5J6T-Z242-20-R18-Z:LED_CUW_Y3SH.B2-GFJD-5J6T-Z242-20-R18-Z, symbol CUW_Y3SH.B2-GFJD-5J6T-Z242-20-R18-Z:CUW_Y3SH.B2-GFJD-5J6T-Z242-20-R18-Z
- added J1: 10118194-0001LF, 10118194-0001LF:AMPHENOL_10118194-0001LF, symbol 10118194-0001LF:10118194-0001LF
- added J2: Conn_01x03_Pin, symbol Connector:Conn_01x03_Pin
- added J3: PRT-14417, qwiic_connector:CONN_PRT-14417_SPK, symbol qwiic_connector:PRT-14417
- added MK1: ICS-43434, Sensor_Audio:InvenSense_ICS-43434-6_3.5x2.65mm, symbol Sensor_Audio:ICS-43434
- added P1: S2B-PH-SM4-TB, S2B-PH-SM4-TB:JST_S2B-PH-SM4-TB, symbol S2B-PH-SM4-TB:S2B-PH-SM4-TB
- added Q1, Q2, Q3: BSD840NH6327XTSA1, BSD840NH6327XTSA1:TRANS_BSD840NH6327XTSA1, symbol BSD840NH6327XTSA1:BSD840NH6327XTSA1
- added R1: 47k, symbol Device:R
- added R10, R3, R4, R5, R6, R7, R8, R9: 120, symbol Device:R
- added R11, R13, R15, R21, R27: 100, symbol Device:R
- added R12, R14, R16, R22, R28: 100k, symbol Device:R
- added R17, R18, R19, R20, R23, R24, R25, R26: 47, symbol Device:R
- added R2: 68, symbol Device:R
- added R29, R30: DNP, symbol Device:R
- added SW1: SW_Push_Dual, symbol Switch:SW_Push_Dual
- added U1: RP2350_Stamp, RP2040_Stamp:RP2040_Stamp_SMD, symbol RP2xxx_Stamp:RP2350_Stamp
- added U2: Common Cathode, custom:SDTC40R2W, symbol custom:SDTC40R2W
- added X1: Badgelife_sao_connector_v169bis, symbol badgelife_shitty_addon_v169bis:Badgelife_sao_connector_v169bis
Connections:
- new net: Q1.6, U2.1 (DIG1)
- new net: Q2.6, U2.10 (DIG2)
- new net: R10.2, U2.11 (F)
- new net: R3.2, U2.2 (DP)
- new net: R4.2, U2.3 (D)
- new net: R5.2, U2.4 (C)
- new net: R6.2, U2.5 (G)
- new net: R7.2, U2.6 (E)
- new net: Q1.3, U2.7 (DIG3)
- new net: R8.2, U2.8 (B)
- new net: R9.2, U2.9 (A)
- new net: D4.A, R20.2
- new net: D1.A, R17.2
- new net: U1.29 (GPIO28), X1.3 (SDA)
- new net: D6.A, R24.2
- new net: D5.C, D6.C, D7.C, D8.C, Q3.3
- new net: D3.A, R19.2
- new net: Q3.5, R27.2, R28.1
- new net: D2.A, R18.2
- new net: D1.C, D2.C, D3.C, D4.C, Q3.6
- new net: Q2.2, R15.2, R16.1
- new net: Q1.2, R11.2, R12.1
- new net: D5.A, R23.2
- new net: D8.A, R26.2
- new net: Q3.2, R21.2, R22.1
- new net: MK1.6 (SD), R1.1, R2.1
- new net: Q1.5, R13.2, R14.1
- new net: D7.A, R25.2
- new net +3.3V: C1.1, C2.1, J3.2, MK1.5 (VDD), R17.1, R18.1, R19.1, R20.1, R23.1, R24.1, R25.1, R26.1, R29.1, R30.1, U1.34 (3.3V), X1.1 (VCC)
- new net +5V: J1.1 (VCC), U1.33 (5V)
- new net 7SEG_A: R9.1, U1.9 (GPIO8)
- new net 7SEG_B: R8.1, U1.8 (GPIO7)
- new net 7SEG_C: R5.1, U1.5 (GPIO4)
- new net 7SEG_D: R4.1, U1.4 (GPIO3)
- new net 7SEG_DIG1: R11.1, U1.11 (GPIO10)
- new net 7SEG_DIG2: R13.1, U1.12 (GPIO11)
- new net 7SEG_DIG3: R15.1, U1.13 (GPIO12)
- new net 7SEG_DP: R3.1, U1.3 (GPIO2)
- new net 7SEG_E: R7.1, U1.7 (GPIO6)
- new net 7SEG_F: R10.1, U1.10 (GPIO9)
- new net 7SEG_G: R6.1, U1.6 (GPIO5)
- new net BCLK: MK1.4 (SCK), U1.19 (GPIO18)
- new net BTN: SW1.1, SW1.3, U1.25 (GPIO24)
- new net DATA: R2.2, U1.21 (GPIO20)
- new net EYE_1: R21.1, U1.17 (GPIO16)
- new net EYE_2: R27.1, U1.18 (GPIO17)
- new net GND: C1.2, C2.2, J1.5 (GND), J1.SH1 (SHIELD), J1.SH2 (SHIELD__1), J1.SH3 (SHIELD__2), J1.SH4 (SHIELD__3), J1.SH5 (SHIELD__4), J1.SH6 (SHIELD__5), J2.2 (Pin_2), J3.1, J3.5 (SH), J3.6 (SH), MK1.2 (LR), MK1.3 (GND), P1.2, Q1.1, Q1.4, Q2.1, Q3.1, Q3.4, R1.2, R12.2, R14.2, R16.2, R22.2, R28.2, SW1.2, SW1.4, U1.31 (GND), X1.2 (GND)
- new net LRCLK: MK1.1 (WS), U1.20 (GPIO19)
- new net QWIIC_SCL: J3.4, R30.2, U1.24 (GPIO23)
- new net QWIIC_SDA: J3.3, R29.2, U1.23 (GPIO22)
- new net SAO_RX: U1.2 (GPIO1), X1.6 (GPIO2)
- new net SAO_SCL: U1.30 (GPIO29), X1.4 (SCL)
- new net SAO_TX: U1.1 (GPIO0), X1.5 (GPIO1)
- new net SWCLK: J2.1 (Pin_1), U1.38 (SWCLK)
- new net SWDIO: J2.3 (Pin_3), U1.37 (SWDIO)
- new net USB_D+: J1.3 (D+), U1.36 (USB_D+)
- new net USB_D-: J1.2 (D-), U1.35 (USB_D-)
- new net VBAT: P1.1, U1.32 (VBAT)
- no-connect marks 0 -> 3
Other:
- note added: "LiPo Battery Connector"
- company: (none) -> creativecommons.org/licenses/by/4.0/
- title: (none) -> Crommeter
