File: hardware/crommeter/crommeter.kicad_sch (KiCad schematic)
At the start: 52 parts, among them J1 10118194-0001LF, J2 Conn_01x03_Pin, J3 PRT-14417, P1 S2B-PH-SM4-TB, Q1 BSD840NH6327XTSA1, Q2 BSD840NH6327XTSA1, Q3 BSD840NH6327XTSA1, SW1 SW_Push_Dual, U1 RP2350_Stamp, U2 Common Cathode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

Commit message: Added artwork
Parts:
- added H1: MountingHole, MountingHole:MountingHole_4.3mm_M4, symbol Mechanical:MountingHole
- added R31: DNP, Resistor_SMD:R_0603_1608Metric_Pad0.98x0.95mm_HandSolder, symbol Device:R
Connections:
- net +3.3V: now also R31.1
- net BTN: now also R31.2
Other:
- moved on the sheet: SW1

Commit message: Added BOM
Parts:
- C1: MANUFACTURER (none) -> YAGEO; Manufacturer Part Number (none) -> CC0603KRX7R7BB104; Part Link (none) -> https://www.digikey.com/en/products/detail/yageo/CC0603KRX7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
- C2: MANUFACTURER (none) -> YAGEO; Manufacturer Part Number (none) -> CC0603KRX7R7BB105; Part Link (none) -> https://www.digikey.com/en/products/detail/yageo/CC0603KRX7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
- D1, D2, D3, D4, D5, D6, D7, D8: Footprint Link (none) -> https://www.digikey.com/en/models/13998110; Manufacturer Part Number (none) -> CUW Y3SH.B2-GFJD-5J6T-Z242-20-R18-Z; Part Link (none) -> https://www.digikey.com/en/products/detail/ams-osram-usa-in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
- J1: Footprint Link (none) -> https://www.digikey.com/en/models/2785389; Manufacturer Part Number (none) -> 10118194-0001LF; Part Link (none) -> https://www.digikey.com/en/products/detail/amphenol-cs-fci/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
- J2: Footprint Link (none) -> https://www.digikey.com/en/models/7916034; MANUFACTURER (none) -> Amphenol ICC (FCI); Manufacturer Part Number (none) -> 10129380-903001BLF; Part Link (none) -> https://www.digikey.com/en/products/detail/amphenol-cs-fci/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
- J3: Footprint Link (none) -> https://www.digikey.com/en/models/7652746; MANUFACTURER (none) -> SparkFun Electronics; Manufacturer Part Number (none) -> 14417; Part Link (none) -> https://www.digikey.com/en/products/detail/sparkfun-electro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
- MK1: Footprint Link (none) -> https://www.digikey.com/en/models/6140298; MANUFACTURER (none) -> TDK InvenSense; Manufacturer Part Number (none) -> ICS-43434; Part Link (none) -> https://www.digikey.com/en/products/detail/tdk-invensense/I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
- P1: Footprint Link (none) -> https://www.digikey.com/en/models/926655; Manufacturer Part Number (none) -> S2B-PH-SM4-TB; Part Link (none) -> https://www.digikey.com/en/products/detail/jst-sales-americ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
- Q1, Q2, Q3: Footprint Link (none) -> https://www.digikey.com/en/models/2783455; Manufacturer Part Number (none) -> BSD840NH6327XTSA1; Part Link (none) -> https://www.digikey.com/en/products/detail/infineon-technol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
- R1: MANUFACTURER (none) -> YAGEO; Manufacturer Part Number (none) -> RC0603FR-0747KL; Part Link (none) -> https://www.digikey.com/en/products/detail/yageo/RC0603FR-0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
- R10, R3, R4, R5, R6, R7, R8, R9: MANUFACTURER (none) -> YAGEO; Manufacturer Part Number (none) -> RC0603JR-7W120RL; Part Link (none) -> https://www.digikey.com/en/products/detail/yageo/RC0603JR-7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
- R11, R13, R15, R21, R27: MANUFACTURER (none) -> YAGEO; Manufacturer Part Number (none) -> RC0603FR-7W100RL; Part Link (none) -> https://www.digikey.com/en/products/detail/yageo/RC0603FR-7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
- R12, R14, R16, R22, R28: MANUFACTURER (none) -> YAGEO; Manufacturer Part Number (none) -> RC0603FR-07100KL; Part Link (none) -> https://www.digikey.com/en/products/detail/yageo/RC0603FR-0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
- R17, R18, R19, R20, R23, R24, R25, R26: MANUFACTURER (none) -> YAGEO; Manufacturer Part Number (none) -> RC0603FR-1347RL; Part Link (none) -> https://www.digikey.com/en/products/detail/yageo/RC0603FR-1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
- R2: MANUFACTURER (none) -> YAGEO; Manufacturer Part Number (none) -> RC0603FR-0768RL; Part Link (none) -> https://www.digikey.com/en/products/detail/yageo/RC0603FR-0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
- SW1: Footprint Link (none) -> https://www.digikey.com/en/models/1201469; MANUFACTURER (none) -> TE Connectivity ALCOSWITCH Switches; Manufacturer Part Number (none) -> FSM2JSMAATR; Part Link (none) -> https://www.digikey.com/en/products/detail/te-connectivity-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
- U1: Footprint Link (none) -> https://github.com/solderparty/rp2xxx_stamp_footprints; MANUFACTURER (none) -> Solder Party; Manufacturer Part Number (none) -> RP2350 Stamp; Part Link (none) -> https://shop.pimoroni.com/products/rp2350-stamp
- U2: MANUFACTURER (none) -> ChromeLED; Manufacturer Part Number (none) -> SDTC40R2W; Part Link (none) -> https://www.digikey.com/en/products/detail/chromeled/SDTC40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
- X1: Footprint Link (none) -> https://cdn.hackaday.io/files/1751827494986688/KiCad_SAOv2.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; MANUFACTURER (none) -> Adam Tech; Manufacturer Part Number (none) -> BHR-06-VUA; Part Link (none) -> https://www.digikey.com/en/products/detail/adam-tech/BHR-06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
