File: hardware/crommeter/crommeter.kicad_pcb (KiCad board)
At the start: 2 copper layers, 53 parts, among them J1 10118194-0001LF, J2 Conn_01x03_Pin, J3 PRT-14417, P1 S2B-PH-SM4-TB, Q1 BSD840NH6327XTSA1, Q2 BSD840NH6327XTSA1, Q3 BSD840NH6327XTSA1, SW1 SW_Push_Dual, U1 RP2350_Stamp, U2 Common Cathode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

Commit message: Added artwork
Parts:
- added G***: LOGO, artwork:cromulon_copper, F.Cu at (127.0, 101.6)
- added G***: LOGO, artwork:cromulon_silkscreen, F.Cu at (127.0, 101.6)
- added G***: LOGO, artwork:cromulon_mask, F.Cu at (127.0, 101.6)
- added H1: MountingHole, MountingHole:MountingHole_4.3mm_M4, F.Cu at (129.5, 44.5)
- moved C1 87.6 mm to (94.0, 91.4), turned to 90 degrees
- moved MK1 86.1 mm to (90.2, 91.4)
- moved C2 85.6 mm to (96.5, 91.4), turned to 90 degrees
- moved R1 84.2 mm to (90.2, 97.8), turned to 0 degrees
- moved R2 79.1 mm to (90.2, 95.2), turned to 0 degrees
- moved R16 75.3 mm to (105.8, 113.0)
- moved R12 72.1 mm to (107.0, 94.0)
- moved R15 71.5 mm to (109.6, 113.0)
- moved R11 67.8 mm to (110.8, 94.0)
- moved R13 67.6 mm to (110.8, 102.9)
- moved R14 65.9 mm to (106.5, 102.9)
- moved Q2 65.4 mm to (107.4, 109.2)
- moved Q1 64.9 mm to (107.4, 97.8)
- moved R10 54.8 mm to (117.2, 104.1)
- moved SW1 54.8 mm to (120.8, 151.9), turned to 90 degrees
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Other:
- board outline added: 83.2 x 125.8 mm
- copper layers 2 -> 4

Commit message: Mostly finished layout
Parts:
- removed the G*** at (127.0, 101.6)
- added G***: LOGO, artwork:cromulon_mask_bot, F.Cu at (127.0, 101.6)
- moved Q1 49.9 mm to (154.9, 113.0), turned to -90 degrees
- moved R14 49.2 mm to (153.7, 116.8)
- moved R11 49.1 mm to (157.5, 109.2)
- moved R12 49.1 mm to (153.7, 109.2)
- moved R13 48.7 mm to (157.5, 116.8)
- moved R15 48.5 mm to (157.5, 105.4)
- moved R16 48.5 mm to (153.7, 105.4)
- moved Q2 48.2 mm to (154.9, 101.6), turned to -90 degrees
- moved J2 27.9 mm to (118.1, 125.7)
- moved R8 27.1 mm to (135.9, 118.7), turned to 90 degrees
- moved R9 24.0 mm to (134.0, 118.7), turned to 90 degrees
- moved R10 20.9 mm to (132.1, 118.7), turned to 90 degrees
- moved R1 15.3 mm to (94.6, 83.2)
- moved R7 12.0 mm to (137.8, 118.7), turned to 90 degrees
- moved R2 11.1 mm to (94.6, 85.1)
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Routing:
- net +3.3V: track 0.00 -> 335.9 mm, vias 0 -> 10
- net /LRCLK: track 0.00 -> 85.0 mm, vias 0 -> 2
- net /BCLK: track 0.00 -> 84.7 mm, vias 0 -> 2
- net /DATA: track 0.00 -> 84.6 mm, vias 0 -> 2
- net Net-(D1-PadC): track 0.00 -> 81.5 mm
- net Net-(D5-PadC): track 0.00 -> 79.8 mm
- net /QWIIC_SDA: track 0.00 -> 73.0 mm
- net /QWIIC_SCL: track 0.00 -> 72.4 mm
- net /EYE_1: track 0.00 -> 69.1 mm, vias 0 -> 2
- net /EYE_2: track 0.00 -> 63.3 mm, vias 0 -> 2
- net Net-(U2-F): track 0.00 -> 41.0 mm
- net /SAO_RX: track 0.00 -> 40.9 mm, vias 0 -> 2
- net /VBAT: track 0.00 -> 38.8 mm, vias 0 -> 4
- net /SAO_TX: track 0.00 -> 38.6 mm, vias 0 -> 2
- net /BTN: track 0.00 -> 38.2 mm
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- added copper zone on B.Cu, net GND
- added copper zone on F.Cu, net GND
Other:
- board text added: "Crommeter"
- board text added: "SHOW ME WHAT YOU GOT!"
- board text added: "WayWayWay"
- board text added: "v01"

Commit message: Generated gerbers
Routing:
- net /VBAT: track 38.8 -> 41.0 mm
- net +3.3V: track 335.9 -> 336.7 mm
Changed lines of the file:
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@@
 		(tenting front back)
 		(pcbplotparams
-			(layerselection 0x00000000_00000000_55555555_5755f5ff)
+			(layerselection 0x00000000_00000000_55555555_5755f5af)
 			(plot_on_all_layers_selection 0x00000000_00000000_00000000_00000000)
 			(disableapertmacros no)
@@
 			(outputformat 1)
 			(mirror no)
-			(drillshape 1)
+			(drillshape 0)
 			(scaleselection 1)
-			(outputdirectory "")
+			(outputdirectory "../gerbers/")
 		)
 	)
@@
 		(net 1)
 	)
+	(segment
+		(start 128.3208 126.238)
+		(end 128.3208 127)
+		(width 1.016)
+		(layer "F.Cu")
+		(net 1)
+	)
 	(via
 		(at 128.3208 143.002)
@@
 		(net 22)
 	)
+	(segment
+		(start 122.8344 140.8938)
+		(end 123.5606 141.62)
+		(width 1.016)
+		(layer "F.Cu")
+		(net 22)
+	)
+	(segment
+		(start 122.0216 131.5974)
+		(end 122.8344 132.4102)
+		(width 1.016)
+		(layer "F.Cu")
+		(net 22)
+	)
 	(via
 		(at 122.8344 140.8938)
@@
 	)
 	(segment
-		(start 130.175 121.0564)
-		(end 130.175 118.2878)
+		(start 129.9464 119.426361)
+		(end 130.175 119.197761)
 		(width 0.2032)
 		(layer "F.Cu")
@@
 	(segment
 		(start 131.5974 122.4788)
-		(end 130.175 121.0564)
+		(end 129.9464 120.8278)
+		(width 0.2032)
+		(layer "F.Cu")
+		(net 54)
+	)
+	(segment
+		(start 130.175 119.197761)
+		(end 130.175 118.2878)
+		(width 0.2032)
+		(layer "F.Cu")
+		(net 54)
+	)
+	(segment
+		(start 129.9464 120.8278)
+		(end 129.9464 119.426361)
 		(width 0.2032)
 		(layer "F.Cu")
